File: PCB/Beanbike-Display.kicad_pcb (KiCad board)
At the start: 2 copper layers, 99.5 x 55.5 mm, 18 parts, among them J1 Conn_01x21_Socket, J2 Conn_01x21_Socket, J5 Conn_01x08_Socket, J6 Conn_01x03_Socket, J7 Conn_01x03_Socket, J8 Conn_01x06_Pin, J9 5034801800, SW1 Up, SW2 Down, SW3 Mode

Commit message: BikeState & RTOS
I forgot to commit
Parts:
- removed R1: 0 Poka Yoke, Resistor_THT:R_Axial_DIN0207_L6.3mm_D2.5mm_P10.16mm_Horizontal
- removed R2: 0 POKA-YOKE, Resistor_THT:R_Axial_DIN0207_L6.3mm_D2.5mm_P10.16mm_Horizontal
- removed SW1: Up, Button_Switch_SMD:SW_SPST_PTS645Sx43SMTR92
- removed SW2: Down, Button_Switch_SMD:SW_SPST_PTS645Sx43SMTR92
- removed SW3: Mode, Button_Switch_SMD:SW_SPST_PTS645Sx43SMTR92
Connections:
- J1 pad 11: GPIO_18 -> unconnected-(J1-Pin_11-Pad11)
- J1 pad 12: GPIO_8 -> unconnected-(J1-Pin_12-Pad12)
- J1 pad 13: GPIO_3 -> unconnected-(J1-Pin_13-Pad13)
- J1 pad 15: unconnected-(J1-Pin_15-Pad15) -> GPIO_9
- J1 pad 16: unconnected-(J1-Pin_16-Pad16) -> GPIO_10
- J2 pad 19: RX -> unconnected-(J2-Pin_19-Pad19)
- J2 pad 20: TX -> unconnected-(J2-Pin_20-Pad20)
- J5 pad 3: Net-(J5-Pin_3) -> GPIO_9
- J5 pad 4: Net-(J5-Pin_4) -> GPIO_10
Routing:
- net GPIO_3: track 69.2 -> 0.00 mm
- net Net-(J5-Pin_4): track 66.8 -> 0.00 mm, vias 2 -> 0
- net GPIO_18: track 66.1 -> 0.00 mm
- net GPIO_8: track 57.6 -> 0.00 mm
- net Net-(J5-Pin_3): track 54.1 -> 0.00 mm, vias 1 -> 0
- net TX: track 24.6 -> 0.00 mm
- net GPIO_9: track 0.00 -> 13.1 mm
- net GPIO_10: track 0.00 -> 13.1 mm
- net RX: track 6.75 -> 0.00 mm
- net GND: vias 38 -> 32
Other:
- board size 99.5 x 55.5 mm -> 83 x 55.5 mm
- board text removed: "Down"
- board text removed: "MODE"
- board text removed: "Up"
